File: main/main.kicad_pcb (KiCad board)
At the start: 4 copper layers, 101.3 x 110 mm, 318 parts, among them J1 3.5mm Jack, J10 3.5mm Jack, J11 3.5mm Jack, J2 3.5mm Jack, J3 3.5mm Jack, J4 3.5mm Jack, J5 3.5mm Jack, J6 2x5 Header, J7 3.5mm Jack, J8 3.5mm Jack, J9 3.5mm Jack, Q1 MMBT3904, Q2 MMBT3904, Q3 MMBT3904, SW1 SW_Rotary8, SW2 SW_Rotary8, SW3 SW_Rotary8, SW4 SW_SPDT, SW5 SW_SPDT, SW6 SW_SPDT, SW7 SW_SPDT, SW8 SW_Rotary8, U1 TL072CP, U10 CD4017, U11 CD4017, U12 4013, U13 4013, U14 CD4046, U15 CD4017, U16 CD40107, U17 CD40107, U18 CD4046, U19 CD4046, U2 AMS1117-5.0, U20 CD4017, U21 CD4017, U22 TL072CP, U23 TL072CP, U24 CD4046, U25 CD4046, U26 CD4017, U27 CD4017, U28 TL072CP, U29 TL072CP, U3 TL072CP, U30 NSL-32SR3, U31 NSL-32SR3, U32 TL072CP, U33 TL072CP, U34 NSL-32SR3, U35 NSL-32SR3, U4 LM317_SOT-223, U5 TL072CP, U6 CD4046, U7 CD4046, U8 CD4046, U9 CD4017

Commit message: Switched PLL cap to 680p
Parts:
- C23: value 1nF -> 680pF
- U12, U13: value 4013 -> CD4013
Changed lines of the file:
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@@
     (at 73.3 140.7 90)
     (descr "http://spec_sheets.e-switch.com/specs/T111597.pdf")
+    (property "Digi-Key Part" "2449-ANT11SF1CQE-ND")
     (property "Sheetfile" "harmonics.kicad_sch")
     (property "Sheetname" "PLLs")
@@
     (at 73.3 74.7 90)
     (descr "http://spec_sheets.e-switch.com/specs/T111597.pdf")
+    (property "Digi-Key Part" "2449-ANT11SF1CQE-ND")
     (property "Sheetfile" "harmonics.kicad_sch")
     (property "Sheetname" "PLLs")
@@
   (footprint "sputterizer:CPA_8" (layer "F.Cu")
     (at 59.7 70)
+    (property "Digi-Key Part" "1528-2925-ND")
     (property "Sheetfile" "harmonics.kicad_sch")
     (property "Sheetname" "PLLs")
@@
     (at 73.3 96.7 90)
     (descr "http://spec_sheets.e-switch.com/specs/T111597.pdf")
+    (property "Digi-Key Part" "2449-ANT11SF1CQE-ND")
     (property "Sheetfile" "harmonics.kicad_sch")
     (property "Sheetname" "PLLs")
@@
   (footprint "sputterizer:CPA_8" (layer "F.Cu")
     (at 59.7 136)
+    (property "Digi-Key Part" "1528-2925-ND")
     (property "Sheetfile" "harmonics.kicad_sch")
     (property "Sheetname" "PLLs")
@@
     (at 73.3 118.7 90)
     (descr "http://spec_sheets.e-switch.com/specs/T111597.pdf")
+    (property "Digi-Key Part" "2449-ANT11SF1CQE-ND")
     (property "Sheetfile" "harmonics.kicad_sch")
     (property "Sheetname" "PLLs")
@@
   (footprint "sputterizer:CPA_8" (layer "F.Cu")
     (at 59.7 92)
+    (property "Digi-Key Part" "1528-2925-ND")
     (property "Sheetfile" "harmonics.kicad_sch")
     (property "Sheetname" "PLLs")
@@
   (footprint "sputterizer:CPA_8" (layer "F.Cu")
     (at 59.7 114)
+    (property "Digi-Key Part" "1528-2925-ND")
     (property "Sheetfile" "harmonics.kicad_sch")
     (property "Sheetname" "PLLs")
@@
     (tags "capacitor handsolder")
     (property "Digi-Key Part" "BC2662CT-ND")
-    (property "LCSC Part #" "C520092")
+    (property "LCSC Part #" "C384742")
     (property "Sheetfile" "harmonics.kicad_sch")
     (property "Sheetname" "PLLs")
@@
     (tags "capacitor handsolder")
     (property "Digi-Key Part" "BC2662CT-ND")
-    (property "LCSC Part #" "C46653")
+    (property "LCSC Part #" "C384742")
     (property "Sheetfile" "harmonics.kicad_sch")
     (property "Sheetname" "PLLs")
@@
       (effects (font (size 0.5 0.5) (thickness 0.1)) (justify mirror))
     )
-    (fp_text value "1nF" (at 0 -1.68 -270) (layer "B.Fab")
+    (fp_text value "680pF" (at 0 -1.68 -270) (layer "B.Fab")
       (effects (font (size 1 1) (thickness 0.15)) (justify mirror))
     )
@@
   (footprint "digikey-footprints:SOIC-14_W3.9mm" (layer "B.Cu")
     (at 72.4 81)
+    (property "Digi-Key Part" "296-24347-1-ND")
+    (property "LCSC Part #" "C13527")
     (property "Sheetfile" "harmonics.kicad_sch")
     (property "Sheetname" "PLLs")
@@
       (effects (font (size 1 1) (thickness 0.15)) (justify mirror))
     )
-    (fp_text value "4013" (at 0 -5.29) (layer "B.Fab")
+    (fp_text value "CD4013" (at 0 -5.29) (layer "B.Fab")
       (effects (font (size 1 1) (thickness 0.15)) (justify mirror))
     )
@@
   (footprint "digikey-footprints:SOIC-14_W3.9mm" (layer "B.Cu")
     (at 72.5 125 180)
+    (property "Digi-Key Part" "296-24347-1-ND")
+    (property "LCSC Part #" "C13527")
     (property "Sheetfile" "harmonics.kicad_sch")
     (property "Sheetname" "PLLs")
@@
       (effects (font (size 1 1) (thickness 0.15)) (justify mirror))
     )
-    (fp_text value "4013" (at 0 -5.29) (layer "B.Fab")
+    (fp_text value "CD4013" (at 0 -5.29) (layer "B.Fab")
       (effects (font (size 1 1) (thickness 0.15)) (justify mirror))
     )
@@
     (tags "capacitor handsolder")
     (property "Digi-Key Part" "BC2662CT-ND")
-    (property "LCSC Part #" "C520092")
+    (property "LCSC Part #" "C384742")
     (property "Sheetfile" "harmonics.kicad_sch")
     (property "Sheetname" "PLLs")
@@
     (tags "capacitor handsolder")
     (property "Digi-Key Part" "BC2662CT-ND")
-    (property "LCSC Part #" "C520092")
+    (property "LCSC Part #" "C384742")
     (property "Sheetfile" "harmonics.kicad_sch")
     (property "Sheetname" "PLLs")

Commit message: Switch to Thonk jacks.
Reduces use of extended parts.
Parts:
- removed H1, H3, H4: MountingHole, MountingHole:MountingHole_2.5mm
- removed H2: locked, MountingHole:MountingHole_2.5mm
- C13, C52, C53, C64, C65, C70, C71, C74, C75: footprint Capacitor_SMD:C_0805_2012Metric_Pad1.18x1.45mm_HandSolder -> Capacitor_SMD:C_0603_1608Metric_Pad1.08x0.95mm_HandSolder
- D10, D11, D12, D13, D14, D17, D18, D19, D20, D21, D22, D23, D24, D5, D6, D7, D8, D9: footprint Diode_SMD:D_0805_2012Metric_Pad1.15x1.40mm_HandSolder -> Diode_SMD:D_SOD-323_HandSoldering
- J1, J10, J11, J2, J3, J4, J5, J7, J8, J9: footprint sputterizer:Molex-0472570001 -> audio jacks:Jack_3.5mm_QingPu_WQP-PJ398SM_Vertical
- U12, U13: footprint digikey-footprints:SOIC-14_W3.9mm -> Package_SO:SOIC-14_3.9x8.7mm_P1.27mm
- moved D21 4.34 mm to (138.6, 128.4), turned to 180 degrees
- moved C46 3.87 mm to (138.8, 125.5)
- moved D15 3.75 mm to (48.1, 46.9), turned to 90 degrees
- moved R2 3.07 mm to (48.0, 134.1), turned to 90 degrees
- moved R4 3.02 mm to (48.0, 112.2), turned to 90 degrees
- moved R1 2.97 mm to (48.0, 90.2), turned to 90 degrees
- moved C23 2.55 mm to (54.5, 62.5)
- moved U34 2.28 mm to (129.1, 130.3)
- moved R36 2.16 mm to (47.9, 65.4), turned to 90 degrees
- moved D16 2.11 mm to (52.8, 51.1), turned to 90 degrees
- moved R48 1.92 mm to (134.7, 128.4), turned to 180 degrees
- moved D22 1.78 mm to (130.8, 128.4), turned to 180 degrees
- moved R3 1.43 mm to (48.0, 69.6), turned to 90 degrees
- moved C26 1.13 mm to (51.5, 64.4)
- moved U7 1.12 mm to (49.6, 60.5)
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Connections:
- R1 pad 2: Net-(J3-Pad2) -> Net-(J3-PadT)
- R2 pad 2: Net-(J5-Pad2) -> Net-(J5-PadT)
- R3 pad 2: Net-(J2-Pad2) -> Net-(J2-PadT)
- R4 pad 2: Net-(J4-Pad2) -> Net-(J4-PadT)
- R44 pad 1: Net-(J8-Pad2) -> Net-(J8-PadT)
- R45 pad 1: Net-(J9-Pad2) -> Net-(J9-PadT)
- R48 pad 1: Net-(J10-Pad2) -> Net-(J10-PadT)
- R49 pad 1: Net-(J11-Pad2) -> Net-(J11-PadT)
- R9 pad 2: Net-(J1-Pad2) -> Net-(J1-PadT)
Routing:
- net GND: track 77.8 -> 58.8 mm
- net Net-(J1-Pad2): track 8.03 -> 0.00 mm, vias 1 -> 0
- net Net-(J1-PadT): track 0.00 -> 7.59 mm, vias 0 -> 1
- net Net-(R35-Pad2): track 5.28 -> 11.0 mm, vias 0 -> 3
- net Net-(J4-Pad2): track 5.58 -> 0.00 mm, vias 1 -> 0
- net Net-(J3-Pad2): track 5.58 -> 0.00 mm, vias 1 -> 0
- net Net-(J5-Pad2): track 5.54 -> 0.00 mm, vias 1 -> 0
- net Net-(J2-PadT): track 0.00 -> 5.18 mm, vias 0 -> 1
- net Net-(D15-Pad1): track 1.81 -> 6.89 mm, vias 0 -> 2
- net +9V: track 237.1 -> 232.0 mm, vias 35 -> 36
- net Net-(J8-PadT): track 0.00 -> 4.96 mm
- net +5V: track 181.0 -> 176.1 mm, vias 10 -> 12
- net Net-(J2-Pad2): track 4.59 -> 0.00 mm
- net Net-(J9-PadT): track 0.00 -> 4.46 mm
- net Net-(J8-Pad2): track 4.45 -> 0.00 mm
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