File: main/main.kicad_sch (KiCad schematic)
At the start: 81 parts, among them J1 3.5mm Jack, J2 3.5mm Jack, J3 3.5mm Jack, J4 3.5mm Jack, J5 3.5mm Jack, J6 2x5 Header, J7 3.5mm Jack, Q2 MMBT3904, Q3 MMBT3906, U1 TL072CP, U3 TL072CP, U4 LM317_SOT-223, U5 TL072CP

Commit message: Latest gain plan.
Version 1.1
Sent to JLCPCB
Parts:
- removed D39, D40: BAT54J, Diode_SMD:D_SOD-323F, symbol Diode:BAT54J
- C7: value 100nF -> 220nF; LCSC Part # C49678 -> C5378
- C8: value 1nF -> 330pF; footprint Capacitor_SMD:C_0805_2012Metric_Pad1.18x1.45mm_HandSolder -> Capacitor_SMD:C_0603_1608Metric_Pad1.08x0.95mm_HandSolder; LCSC Part # C62774 -> C1664
- J6: LCSC Part # C124391 -> C19268827
- R13: value 91K -> 88.7K; LCSC Part # C23265 -> C163418
- R19: value 10K -> 5.1K; LCSC Part # C25804 -> C23186
- RV1: footprint sputterizer:HDK_3mm -> Potentiometer_SMD:Potentiometer_Bourns_3224W_Vertical; Digi-Key Part 118-TC33X-1-501ECT-ND -> (none); LCSC Part # C720649 -> C116324
Other:
- removed sheet Hi Pass Filters
- moved on the sheet: C10, C11, C14, R18, R21, RV1, TP24, U4

Commit message: Version 1.2
Parts:
- C12: value 100pF -> 2.7nF; LCSC Part # C1790 -> C97900
- C13: value 10pF -> 2nF; LCSC Part # C1634 -> C2168932
- C17: value 1nF -> 2.7nF; LCSC Part # C62774 -> C97900
- C20: value 100pF -> 270pF; LCSC Part # C1790 -> C527216
- R17: value 133K -> 7.87K; LCSC Part # C321714 -> C103822
- R20: value 475K -> 16.5K; LCSC Part # C403244 -> C227613
- R23: value 4.7K -> 16.5K; LCSC Part # C23162 -> C227613
- R26: value 143K -> 59K; LCSC Part # C304703 -> C218088
Other:
- note added: "Low-Pass; 4th order Butterworth 5kHz passband"
- note removed: "Low-Pass; 4th order Butterworth 20kHz passband"

Commit message: v2.0
Parts:
- J1, J2, J3, J4, J5, J7: footprint audio jacks:Jack_3.5mm_QingPu_WQP-PJ398SM_Vertical -> greenface:Jack_3.5mm_QingPu_WQP-PJ398SM_Vertical
- RV1: footprint Potentiometer_SMD:Potentiometer_Bourns_3224W_Vertical -> greenface:Trimpot_3.8mmx3.6mm_TC33X-2-103E; symbol dk_Trimmer-Potentiometers:TC33X-2-103E -> greenface:TC33X-2-103E; Category (none) -> Potentiometers, Variable Resistors; DK_Datasheet_Link (none) -> https://www.bourns.com/docs/Product-Datasheets/TC33.pdf; DK_Detail_Page (none) -> /product-detail/en/bourns-inc/TC33X-2-103E/TC33X-103ETR-ND/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; Description_1 (none) -> TRIMMER 10K OHM 0.1W J LEAD TOP; Digi-Key_PN (none) -> TC33X-103ETR-ND; Family (none) -> Trimmer Potentiometers; MPN (none) -> TC33X-2-103E; Manufacturer (none) -> Bourns Inc.; Status (none) -> Active
Connections:
- net SIG: now reaches C17.1, D21.3, R28.1, U5.1, U5.2 (-)
Other:
- note added: "Low-Pass; 4th order Butterworth 5kHz passband Possibly use: mcp6071"
- note removed: "Low-Pass; 4th order Butterworth 5kHz passband"
