File: main/parts.kicad_sch (KiCad schematic)
At the start: 35 parts, among them J12 Eurorack Power Cable

Commit message: Version 1.0
Parts:
- removed GR1: small_logo, panel:small_face, symbol greenface-symbols:small_logo
- removed GR2: big face, panel:face_logo, symbol greenface-symbols:small_logo
- removed N1, N2, N3, N4: Nut, symbol Mechanical:MountingHole
- removed SC1, SC3, SC5, SC7: Nylon Screw, symbol Mechanical:MountingHole
- removed SO6, SO8: Standoff 15mm, symbol Mechanical:MountingHole
- removed SO7: Standoff 12mm, symbol Mechanical:MountingHole
- SO1, SO3, SO5: value Standoff 12mm -> LED Spacer 9mm; Digi-Key Part 732-13063-ND -> RPC4262-ND
- SO2, SO4: value Standoff 15mm -> LED Spacer 9mm; Digi-Key Part 732-13072-ND -> RPC4262-ND
Other:
- note added: "Knobs"
- note added: "LED Spacers"
- note removed: "For attaching board to panel"
- note removed: "For attaching sub-board to panel"
- moved on the sheet: KN1, KN2, KN3, KN4, KN5, KN6, KN7, KN8, SC2, SC4, SC6, SC8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

Commit message: Work in progress
Adds User Manual
Changes CV range to 0 - 8V
Adds spice vactrol test circuit.
Adds VCA spice study
Updates other spice and excel files.
Other:
- title: (none) -> Twangilizer
Changed lines of the file:
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@@
   (paper "A4")
   (title_block
-    (rev "1.0")
+    (title "Twangilizer")
+    (rev "1.1")
   )
   (text "For attaching module to rack" (at 62.23 33.655 0)
