File: main/wavegen.kicad_sch (KiCad schematic)
At the start: 102 parts, among them U18 CD4046, U19 CD4046, U20 CD4017, U21 CD4017, U22 TL072CP, U23 TL072CP, U24 CD4046, U25 CD4046, U26 CD4017, U27 CD4017

Commit message: Latest gain plan.
Version 1.1
Sent to JLCPCB
Parts:
- added TP12: TestPoint, TestPoint:TestPoint_Loop_D2.54mm_Drill1.5mm_Beaded, symbol Connector:TestPoint
- C52, C53, C70, C71: value 300pF -> 1nF; LCSC Part # C519401 -> C1588
- RV6, RV7, RV8, RV9: LCSC Part # C145161 -> C913246
Connections:
- net VC2: now also TP12.1
Changed lines of the file:
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@@
     (stroke (width 0) (type default) (color 0 0 0 0))
   )
+  (wire (pts (xy 196.85 69.85) (xy 193.675 69.85))
+    (stroke (width 0) (type default) (color 0 0 0 0))
+  )
   (wire (pts (xy 137.16 19.05) (xy 137.16 29.845))
     (stroke (width 0) (type default) (color 0 0 0 0))
@@
     (stroke (width 0) (type default) (color 0 0 0 0))
   )
+  (wire (pts (xy 196.85 66.675) (xy 196.85 69.85))
+    (stroke (width 0) (type default) (color 0 0 0 0))
+  )
   (wire (pts (xy 191.77 116.205) (xy 191.77 117.475))
     (stroke (width 0) (type default) (color 0 0 0 0))
@@
     )
   )
+  (global_label "VC2" (shape input) (at 193.675 69.85 180) (fields_autoplaced)
+    (effects (font (size 1.27 1.27)) (justify right))
+    (property "Intersheet References" "${INTERSHEET_REFS}" (id 0) (at 187.6938 69.9294 0)
+      (effects (font (size 1.27 1.27)) (justify right) hide)
+    )
+  )
   (global_label "OSC3" (shape output) (at 141.605 107.95 0) (fields_autoplaced)
     (effects (font (size 1.27 1.27)) (justify left))
@@
       (effects (font (size 1.27 1.27)) (justify left))
     )
-    (property "Value" "300pF" (id 1) (at 151.765 111.76 0)
+    (property "Value" "1nF" (id 1) (at 151.765 111.76 0)
       (effects (font (size 1.27 1.27)) (justify left))
     )
@@
       (effects (font (size 1.27 1.27)) hide)
     )
-    (property "LCSC Part #" "C519401" (id 5) (at 156.845 109.22 0)
+    (property "LCSC Part #" "C1588" (id 5) (at 156.845 109.22 0)
       (effects (font (size 1.27 1.27)) hide)
     )
@@
       (effects (font (size 1.27 1.27)) hide)
     )
-    (property "LCSC Part #" "C145161" (id 6) (at 18.415 63.5 0)
+    (property "LCSC Part #" "C913246" (id 6) (at 18.415 63.5 0)
       (effects (font (size 1.27 1.27)) hide)
     )
@@
       (effects (font (size 1.27 1.27)) hide)
     )
-    (property "LCSC Part #" "C145161" (id 6) (at 18.415 132.715 0)
+    (property "LCSC Part #" "C913246" (id 6) (at 18.415 132.715 0)
       (effects (font (size 1.27 1.27)) hide)
     )
@@
       (effects (font (size 1.27 1.27)) hide)
     )
-    (property "LCSC Part #" "C145161" (id 6) (at 156.845 132.715 0)
+    (property "LCSC Part #" "C913246" (id 6) (at 156.845 132.715 0)
       (effects (font (size 1.27 1.27)) hide)
     )
@@
       (effects (font (size 1.27 1.27)) (justify left))
     )
-    (property "Value" "300pF" (id 1) (at 13.335 111.76 0)
+    (property "Value" "1nF" (id 1) (at 13.335 111.76 0)
       (effects (font (size 1.27 1.27)) (justify left))
     )
@@
       (effects (font (size 1.27 1.27)) hide)
     )
-    (property "LCSC Part #" "C519401" (id 5) (at 18.415 109.22 0)
+    (property "LCSC Part #" "C1588" (id 5) (at 18.415 109.22 0)
       (effects (font (size 1.27 1.27)) hide)
     )
@@
       (effects (font (size 1.27 1.27)) (justify left))
     )
-    (property "Value" "300pF" (id 1) (at 151.13 41.275 0)
+    (property "Value" "1nF" (id 1) (at 151.13 41.275 0)
       (effects (font (size 1.27 1.27)) (justify left))
     )
@@
       (effects (font (size 1.27 1.27)) hide)
     )
-    (property "LCSC Part #" "C519401" (id 5) (at 156.21 38.735 0)
+    (property "LCSC Part #" "C1588" (id 5) (at 156.21 38.735 0)
       (effects (font (size 1.27 1.27)) hide)
     )
@@
     (pin "7")
   )
+  (symbol (lib_id "Connector:TestPoint") (at 196.85 66.675 0) (unit 1)
+    (in_bom yes) (on_board yes)
+    (property "Reference" "TP12" (id 0) (at 198.3232 63.6778 0)
+      (effects (font (size 1.27 1.27)) (justify left))
+    )
+    (property "Value" "TestPoint" (id 1) (at 198.3232 65.9892 0)
+      (effects (font (size 1.27 1.27)) (justify left) hide)
+    )
+    (property "Footprint" "TestPoint:TestPoint_Loop_D2.54mm_Drill1.5mm_Beaded" (id 2) (at 201.93 66.675 0)
+      (effects (font (size 1.27 1.27)) hide)
+    )
+    (property "Datasheet" "~" (id 3) (at 201.93 66.675 0)
+      (effects (font (size 1.27 1.27)) hide)
+    )
+    (property "Digi-Key Part" "36-5006-ND" (id 4) (at 196.85 66.675 0)
+      (effects (font (size 1.27 1.27)) hide)
+    )
+    (property "LCSC Part #" "C5199801" (id 5) (at 196.85 66.675 0)
+      (effects (font (size 1.27 1.27)) hide)
+    )
+    (pin "1")
+  )
   (symbol (lib_id "power:GND") (at 215.265 65.405 0) (unit 1)
     (in_bom yes) (on_board yes)
@@
       (effects (font (size 1.27 1.27)) (justify left))
     )
-    (property "Value" "300pF" (id 1) (at 13.335 41.275 0)
+    (property "Value" "1nF" (id 1) (at 13.335 41.275 0)
       (effects (font (size 1.27 1.27)) (justify left))
     )
@@
       (effects (font (size 1.27 1.27)) hide)
     )
-    (property "LCSC Part #" "C519401" (id 5) (at 18.415 38.735 0)
+    (property "LCSC Part #" "C1588" (id 5) (at 18.415 38.735 0)
       (effects (font (size 1.27 1.27)) hide)
     )
@@
       (effects (font (size 1.27 1.27)) hide)
     )
-    (property "LCSC Part #" "C145161" (id 6) (at 156.21 63.5 0)
+    (property "LCSC Part #" "C913246" (id 6) (at 156.21 63.5 0)
       (effects (font (size 1.27 1.27)) hide)
     )

Commit message: Version 1.2
Parts:
- C52, C53, C70, C71: value 1nF -> 2.2fF; LCSC Part # C1588 -> C1604
- C56, C57, C72, C73: value 10uF -> 4.7uF; LCSC Part # C15850 -> C1779
- R100, R106, R70, R72: LCSC Part # C861179 -> C321771
Changed lines of the file:
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@@
   (title_block
     (title "Twangilizer")
-    (rev "1.1")
+    (rev "1.2")
   )
   (junction (at 81.915 187.96) (diameter 0) (color 0 0 0 0)
@@
       (effects (font (size 1.27 1.27)) (justify left))
     )
-    (property "Value" "10uF" (id 1) (at 193.675 120.65 0)
+    (property "Value" "4.7uF" (id 1) (at 193.675 120.65 0)
       (effects (font (size 1.27 1.27)) (justify left))
     )
@@
       (effects (font (size 1.27 1.27)) hide)
     )
-    (property "LCSC Part #" "C15850" (id 5) (at 191.77 120.015 0)
+    (property "LCSC Part #" "C1779" (id 5) (at 191.77 120.015 0)
       (effects (font (size 1.27 1.27)) hide)
     )
@@
       (effects (font (size 1.27 1.27)) (justify left))
     )
-    (property "Value" "10uF" (id 1) (at 55.245 120.65 0)
+    (property "Value" "4.7uF" (id 1) (at 55.245 120.65 0)
       (effects (font (size 1.27 1.27)) (justify left))
     )
@@
       (effects (font (size 1.27 1.27)) hide)
     )
-    (property "LCSC Part #" "C15850" (id 5) (at 53.34 120.015 0)
+    (property "LCSC Part #" "C1779" (id 5) (at 53.34 120.015 0)
       (effects (font (size 1.27 1.27)) hide)
     )
@@
       (effects (font (size 1.27 1.27)) (justify left))
     )
-    (property "Value" "10uF" (id 1) (at 193.04 50.165 0)
+    (property "Value" "4.7uF" (id 1) (at 193.04 50.165 0)
       (effects (font (size 1.27 1.27)) (justify left))
     )
@@
       (effects (font (size 1.27 1.27)) hide)
     )
-    (property "LCSC Part #" "C15850" (id 5) (at 191.135 49.53 0)
+    (property "LCSC Part #" "C1779" (id 5) (at 191.135 49.53 0)
       (effects (font (size 1.27 1.27)) hide)
     )
@@
       (effects (font (size 1.27 1.27)) hide)
     )
-    (property "LCSC Part #" "C861179" (id 5) (at 243.205 123.19 0)
+    (property "LCSC Part #" "C321771" (id 5) (at 243.205 123.19 0)
       (effects (font (size 1.27 1.27)) hide)
     )
@@
       (effects (font (size 1.27 1.27)) (justify left))
     )
-    (property "Value" "1nF" (id 1) (at 151.765 111.76 0)
+    (property "Value" "2.2fF" (id 1) (at 151.765 111.76 0)
       (effects (font (size 1.27 1.27)) (justify left))
     )
@@
       (effects (font (size 1.27 1.27)) hide)
     )
-    (property "LCSC Part #" "C1588" (id 5) (at 156.845 109.22 0)
+    (property "LCSC Part #" "C1604" (id 5) (at 156.845 109.22 0)
       (effects (font (size 1.27 1.27)) hide)
     )
@@
       (effects (font (size 1.27 1.27)) hide)
     )
-    (property "LCSC Part #" "C861179" (id 5) (at 105.41 52.705 0)
+    (property "LCSC Part #" "C321771" (id 5) (at 105.41 52.705 0)
       (effects (font (size 1.27 1.27)) hide)
     )
@@
       (effects (font (size 1.27 1.27)) (justify left))
     )
-    (property "Value" "1nF" (id 1) (at 13.335 111.76 0)
+    (property "Value" "2.2fF" (id 1) (at 13.335 111.76 0)
       (effects (font (size 1.27 1.27)) (justify left))
     )
@@
       (effects (font (size 1.27 1.27)) hide)
     )
-    (property "LCSC Part #" "C1588" (id 5) (at 18.415 109.22 0)
+    (property "LCSC Part #" "C1604" (id 5) (at 18.415 109.22 0)
       (effects (font (size 1.27 1.27)) hide)
     )
@@
       (effects (font (size 1.27 1.27)) (justify left))
     )
-    (property "Value" "1nF" (id 1) (at 151.13 41.275 0)
+    (property "Value" "2.2fF" (id 1) (at 151.13 41.275 0)
       (effects (font (size 1.27 1.27)) (justify left))
     )
@@
       (effects (font (size 1.27 1.27)) hide)
     )
-    (property "LCSC Part #" "C1588" (id 5) (at 156.21 38.735 0)
+    (property "LCSC Part #" "C1604" (id 5) (at 156.21 38.735 0)
       (effects (font (size 1.27 1.27)) hide)
     )
@@
       (effects (font (size 1.27 1.27)) hide)
     )
-    (property "LCSC Part #" "C861179" (id 5) (at 105.41 123.19 0)
+    (property "LCSC Part #" "C321771" (id 5) (at 105.41 123.19 0)
       (effects (font (size 1.27 1.27)) hide)
     )
@@
       (effects (font (size 1.27 1.27)) hide)
     )
-    (property "LCSC Part #" "C861179" (id 5) (at 243.205 52.705 0)
+    (property "LCSC Part #" "C321771" (id 5) (at 243.205 52.705 0)
       (effects (font (size 1.27 1.27)) hide)
     )
@@
       (effects (font (size 1.27 1.27)) (justify left))
     )
-    (property "Value" "10uF" (id 1) (at 55.245 50.165 0)
+    (property "Value" "4.7uF" (id 1) (at 55.245 50.165 0)
       (effects (font (size 1.27 1.27)) (justify left))
     )
@@
       (effects (font (size 1.27 1.27)) hide)
     )
-    (property "LCSC Part #" "C15850" (id 5) (at 53.34 49.53 0)
+    (property "LCSC Part #" "C1779" (id 5) (at 53.34 49.53 0)
       (effects (font (size 1.27 1.27)) hide)
     )
@@
       (effects (font (size 1.27 1.27)) (justify left))
     )
-    (property "Value" "1nF" (id 1) (at 13.335 41.275 0)
+    (property "Value" "2.2fF" (id 1) (at 13.335 41.275 0)
       (effects (font (size 1.27 1.27)) (justify left))
     )
@@
       (effects (font (size 1.27 1.27)) hide)
     )
-    (property "LCSC Part #" "C1588" (id 5) (at 18.415 38.735 0)
+    (property "LCSC Part #" "C1604" (id 5) (at 18.415 38.735 0)
       (effects (font (size 1.27 1.27)) hide)
     )

Commit message: v2.0
Parts:
- C52, C53, C70, C71: value 2.2fF -> 2.2nF
- RV6, RV7, RV8, RV9: footprint sputterizer:HDK_3mm -> greenface:Trimpot_3.8mmx3.6mm_TC33X-2-103E; symbol dk_Trimmer-Potentiometers:TC33X-2-103E -> greenface:TC33X-2-103E; Category (none) -> Potentiometers, Variable Resistors; DK_Datasheet_Link (none) -> https://www.bourns.com/docs/Product-Datasheets/TC33.pdf; DK_Detail_Page (none) -> /product-detail/en/bourns-inc/TC33X-2-103E/TC33X-103ETR-ND/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; Description_1 (none) -> TRIMMER 10K OHM 0.1W J LEAD TOP; Digi-Key_PN (none) -> TC33X-103ETR-ND; Family (none) -> Trimmer Potentiometers; MPN (none) -> TC33X-2-103E; Manufacturer (none) -> Bourns Inc.; Status (none) -> Active
