File: panel/panel.kicad_pcb (KiCad board)
At the start: 2 copper layers, 101.3 x 128.4 mm, 42 parts

Commit message: Switch to Thonk jacks.
Reduces use of extended parts.
Parts:
- removed H17, H18, H19, H20: MountingHole, MountingHole:MountingHole_2.5mm
- H10, H11, H12, H13, H14, H21, H6, H7, H8, H9: footprint panel:MolexJack -> panel:Jack_3.5mm_QingPu_WQP-PJ398SM_Vertical
- moved H10 0.88 mm to (45.4, 70.0), turned to 0 degrees
- moved H11 0.88 mm to (45.4, 92.0), turned to 0 degrees
- moved H12 0.88 mm to (45.4, 114.0), turned to 0 degrees
- moved H21 0.88 mm to (45.4, 136.0), turned to 0 degrees
- moved H6 0.88 mm to (45.4, 50.0), turned to 180 degrees
- moved H13 0.87 mm to (136.0, 114.0), turned to 0 degrees
- moved H14 0.87 mm to (136.0, 136.0), turned to 0 degrees
- moved H8 0.87 mm to (136.0, 70.0), turned to 0 degrees
- moved H9 0.87 mm to (136.0, 92.0), turned to 0 degrees
- moved H7 0.87 mm to (136.0, 50.0), turned to 0 degrees
- moved H15 0.20 mm to (59.9, 70.0)
- moved H29 0.20 mm to (59.9, 92.0)
- moved H30 0.20 mm to (59.9, 114.0)
- moved H31 0.20 mm to (59.9, 136.0)

Commit message: Version 1.0
Parts:
- removed GR7: face, panel:small_face
- GR3: value bamboo -> Vibrations
- H1, H2, H3, H4: footprint panel:MountingHole_3.2mm_M3_SmPad -> panel:MountingHole_3.2mm_M3_Slot
- moved GR3 7.00 mm to (90.7, 98.0)
Other:
- board text added: "5V Sq."
- board text added: "ANALOG OUT"
- board text added: "CLOCK IN"
- board text added: "Sync Out"
- board text added: "The Twangilizer"
- board text removed: "1f"
- board text removed: "2f"
- board text removed: "3f"
- board text removed: "4f"
- board text removed: "5"
- board text removed: "5f"
- board text removed: "6"
- board text removed: "6f"
- board text removed: "7"
- board text removed: "7f"
- board text removed: "8"
- board text removed: "8f"
- board text removed: "> .1Vp-p"
- board text removed: "Analog"
- board text removed: "Argh Ptoo"
- board text removed: "CLK In"
- board text removed: "Level"
- board text removed: "Out"
- board text removed: "Output"
- board text removed: "Outputs"
- board text removed: "{dblquote}The Twangilizer{dblquote}"
