File: panel/panel.kicad_sch (KiCad schematic)
At the start: 42 parts

Commit message: Switch to Thonk jacks.
Reduces use of extended parts.
Parts:
- removed H17, H18, H19, H20: MountingHole, MountingHole:MountingHole_2.5mm, symbol Mechanical:MountingHole
- H10, H11, H12, H13, H14, H21, H6, H7, H8, H9: footprint panel:MolexJack -> panel:Jack_3.5mm_QingPu_WQP-PJ398SM_Vertical
Other:
- note removed: "Sub Board"
- moved on the sheet: H16, H22, H23, H24, H25, H26, H27, H28, H5

Commit message: Version 1.0
Parts:
- GR3: value bamboo -> Vibrations
- H1, H2, H3, H4: footprint panel:MountingHole_3.2mm_M3_SmPad -> panel:MountingHole_3.2mm_M3_Slot
Other:
- moved on the sheet: GR2, GR3
Changed lines of the file:
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@@
     )
   )
-  (symbol (lib_id "Graphic:Logo_Open_Hardware_Small") (at 256.54 119.38 0) (unit 1)
-    (in_bom yes) (on_board yes)
-    (property "Reference" "GR2" (id 0) (at 256.54 112.395 0))
-    (property "Value" "Logo_Open_Hardware_Small" (id 1) (at 256.54 125.095 0)
-      (effects (font (size 1.27 1.27)) hide)
-    )
-    (property "Footprint" "Symbol:OSHW-Logo_5.7x6mm_SilkScreen" (id 2) (at 256.54 119.38 0)
-      (effects (font (size 1.27 1.27)) hide)
-    )
-    (property "Datasheet" "~" (id 3) (at 256.54 119.38 0)
+  (symbol (lib_id "Graphic:Logo_Open_Hardware_Small") (at 260.985 136.525 0) (unit 1)
+    (in_bom yes) (on_board yes)
+    (property "Reference" "GR2" (id 0) (at 260.985 129.54 0))
+    (property "Value" "Logo_Open_Hardware_Small" (id 1) (at 260.985 142.24 0)
+      (effects (font (size 1.27 1.27)) hide)
+    )
+    (property "Footprint" "Symbol:OSHW-Logo_5.7x6mm_SilkScreen" (id 2) (at 260.985 136.525 0)
+      (effects (font (size 1.27 1.27)) hide)
+    )
+    (property "Datasheet" "~" (id 3) (at 260.985 136.525 0)
       (effects (font (size 1.27 1.27)) hide)
     )
@@
       (effects (font (size 1.27 1.27)) (justify left))
     )
-    (property "Footprint" "panel:MountingHole_3.2mm_M3_SmPad" (id 2) (at 36.83 118.745 0)
+    (property "Footprint" "panel:MountingHole_3.2mm_M3_Slot" (id 2) (at 36.83 118.745 0)
       (effects (font (size 1.27 1.27)) hide)
     )
@@
       (effects (font (size 1.27 1.27)) (justify left))
     )
-    (property "Footprint" "panel:MountingHole_3.2mm_M3_SmPad" (id 2) (at 36.83 145.415 0)
+    (property "Footprint" "panel:MountingHole_3.2mm_M3_Slot" (id 2) (at 36.83 145.415 0)
       (effects (font (size 1.27 1.27)) hide)
     )
@@
       (effects (font (size 1.27 1.27)) (justify left))
     )
-    (property "Footprint" "panel:MountingHole_3.2mm_M3_SmPad" (id 2) (at 36.83 127.635 0)
+    (property "Footprint" "panel:MountingHole_3.2mm_M3_Slot" (id 2) (at 36.83 127.635 0)
       (effects (font (size 1.27 1.27)) hide)
     )
@@
   )
   (symbol (lib_id "greenface-symbols:small_logo") (at 259.08 80.645 0) (unit 1)
-    (in_bom yes) (on_board yes) (fields_autoplaced)
+    (in_bom yes) (on_board no) (fields_autoplaced)
     (property "Reference" "GR7" (id 0) (at 259.08 75.5355 0))
     (property "Value" "face" (id 1) (at 259.08 78.3106 0))
@@
     )
   )
-  (symbol (lib_id "greenface-symbols:small_logo") (at 257.81 139.7 0) (unit 1)
+  (symbol (lib_id "greenface-symbols:small_logo") (at 260.35 117.475 0) (unit 1)
     (in_bom yes) (on_board yes) (fields_autoplaced)
-    (property "Reference" "GR3" (id 0) (at 257.81 134.5905 0))
-    (property "Value" "bamboo" (id 1) (at 257.81 137.3656 0))
-    (property "Footprint" "panel:vib" (id 2) (at 257.81 139.7 0)
-      (effects (font (size 1.27 1.27)) hide)
-    )
-    (property "Datasheet" "" (id 3) (at 257.81 139.7 0)
+    (property "Reference" "GR3" (id 0) (at 260.35 112.3655 0))
+    (property "Value" "Vibrations" (id 1) (at 260.35 115.1406 0))
+    (property "Footprint" "panel:vib" (id 2) (at 260.35 117.475 0)
+      (effects (font (size 1.27 1.27)) hide)
+    )
+    (property "Datasheet" "" (id 3) (at 260.35 117.475 0)
       (effects (font (size 1.27 1.27)) hide)
     )
@@
       (effects (font (size 1.27 1.27)) (justify left))
     )
-    (property "Footprint" "panel:MountingHole_3.2mm_M3_SmPad" (id 2) (at 36.83 136.525 0)
+    (property "Footprint" "panel:MountingHole_3.2mm_M3_Slot" (id 2) (at 36.83 136.525 0)
       (effects (font (size 1.27 1.27)) hide)
     )
@@
     )
     (path "/bd6f6aaa-569a-4c75-a8ff-b09aedaec1f5"
-      (reference "GR3") (unit 1) (value "bamboo") (footprint "panel:vib")
+      (reference "GR3") (unit 1) (value "Vibrations") (footprint "panel:vib")
     )
     (path "/15a85bee-d62c-4957-9712-4492ffd668aa"
@@
     )
     (path "/495b9f3e-72d4-4443-8d1b-2b95612acb36"
-      (reference "H1") (unit 1) (value "MountingHole_Pad") (footprint "panel:MountingHole_3.2mm_M3_SmPad")
+      (reference "H1") (unit 1) (value "MountingHole_Pad") (footprint "panel:MountingHole_3.2mm_M3_Slot")
     )
     (path "/9d5ddb59-1e9e-4537-9599-057acace239b"
-      (reference "H2") (unit 1) (value "MountingHole_Pad") (footprint "panel:MountingHole_3.2mm_M3_SmPad")
+      (reference "H2") (unit 1) (value "MountingHole_Pad") (footprint "panel:MountingHole_3.2mm_M3_Slot")
     )
     (path "/f2be02da-9018-4a96-8543-13b5296b0ced"
-      (reference "H3") (unit 1) (value "MountingHole_Pad") (footprint "panel:MountingHole_3.2mm_M3_SmPad")
+      (reference "H3") (unit 1) (value "MountingHole_Pad") (footprint "panel:MountingHole_3.2mm_M3_Slot")
     )
     (path "/5c470add-b449-455e-95fc-baae46d35c85"
-      (reference "H4") (unit 1) (value "MountingHole_Pad") (footprint "panel:MountingHole_3.2mm_M3_SmPad")
+      (reference "H4") (unit 1) (value "MountingHole_Pad") (footprint "panel:MountingHole_3.2mm_M3_Slot")
     )
     (path "/bcb71876-c270-45b1-942b-f8b7b2e74527"

Commit message: v2.0
Parts:
- added H17: MountingHole, panel:3mmLED, symbol Mechanical:MountingHole
